Commit message: fixed typo

File: catkin_ws/src/my_robot/urdf/my_robot.xacro (robot description, xacro)
@@ -1,4 +1,5 @@
 <?xml version='1.0'?>
-<robot name="my_robot" xmlns:xacro="http://www.ros.org/wiki/xacro">
+<robot name="my_robot"
+  xmlns:xacro="http://www.ros.org/wiki/xacro">
   <link name="robot_footprint"></link>
   <joint name="robot_footprint_joint" type="fixed">
@@ -12,9 +13,5 @@
       <mass value="15.0"/>
       <origin xyz="0.0 0 0" rpy=" 0 0 0"/>
-      <inertia
-          ixx="0.1" ixy="0" ixz="0"
-          iyy="0.1" iyz="0"
-          izz="0.1"
-      />
+      <inertia ixx="0.1" ixy="0" ixz="0" iyy="0.1" iyz="0" izz="0.1" />
     </inertial>
     <collision name='collision'>
@@ -55,49 +52,43 @@
     </visual>
   </link>
-   <link name='left_wheel'>
-	<geometry>
-		<cyclinder radius="0.1" length="0.05">
-	</geometry>
-	<origin>
-	<inertial>
-   		<origin xyz="0 0 0" rpy="0 1.5707 1.5707""/>
-        	<mass value="5"/>
-	<inertia>
-		ixx="0.1" ixy="0" ixz="0"
-    		iyy="0.1" iyz="0"
-    		izz="0.1"
-	</inertia>
-	</internal>
-  </link>
-   <link name='right_wheel'>
-	<geometry>
-		<cyclinder radius="0.1" length="0.05">
-	</geometry>
-	<origin>
-	<inertial>
-   		<origin xyz="0 0 0" rpy="0 1.5707 1.5707""/>
-        	<mass value="5"/>
-	<inertia>
-		ixx="0.1" ixy="0" ixz="0"
-    		iyy="0.1" iyz="0"
-    		izz="0.1"
-	</inertia>
-	</internal>
-	</link>
-<joint type="continuous" name="left_wheel_hinge">
-    <origin xyz="0 0.15 0" rpy="0 0 0"/>
-    <child link="left_wheel"/>
-    <parent link="chassis"/>
-    <axis xyz="0 1 0" rpy="0 0 0"/>
-    <limit effort="10000" velocity="1000"/>
-    <dynamics damping="1.0" friction="1.0"/>
-  </joint>
-<joint type="continuous" name="right_wheel_hinge">
-    <origin xyz="0 0.15 0" rpy="0 0 0"/>
-    <child link="right_wheel"/>
-    <parent link="chassis"/>
-    <axis xyz="0 1 0" rpy="0 0 0"/>
-    <limit effort="10000" velocity="1000"/>
-    <dynamics damping="1.0" friction="1.0"/>
-  </joint>
-</robot>
+  <link name='left_wheel'>
+    <geometry>
+      <cyclinder radius="0.1" length="0.05">
+      </geometry>
+      <origin>
+        <inertial>
+          <origin xyz="0 0 0" rpy="0 1.5707 1.5707"/>
+<mass value="5"/>
+          <inertia> ixx="0.1" ixy="0" ixz="0" iyy="0.1" iyz="0" izz="0.1"
+          </inertia>
+        </internal>
+      </link>
+      <link name='right_wheel'>
+        <geometry>
+          <cyclinder radius="0.1" length="0.05">
+          </geometry>
+          <origin>
+            <inertial>
+              <origin xyz="0 0 0" rpy="0 1.5707 1.5707"/>
+              <mass value="5"/>
+              <inertia> ixx="0.1" ixy="0" ixz="0" iyy="0.1" iyz="0" izz="0.1"
+              </inertia>
+            </inertial>
+          </link>
+          <joint type="continuous" name="left_wheel_hinge">
+            <origin xyz="0 0.15 0" rpy="0 0 0"/>
+            <child link="left_wheel"/>
+            <parent link="chassis"/>
+            <axis xyz="0 1 0" rpy="0 0 0"/>
+            <limit effort="10000" velocity="1000"/>
+            <dynamics damping="1.0" friction="1.0"/>
+          </joint>
+          <joint type="continuous" name="right_wheel_hinge">
+            <origin xyz="0 0.15 0" rpy="0 0 0"/>
+            <child link="right_wheel"/>
+            <parent link="chassis"/>
+            <axis xyz="0 1 0" rpy="0 0 0"/>
+            <limit effort="10000" velocity="1000"/>
+            <dynamics damping="1.0" friction="1.0"/>
+          </joint>
+        </robot>

Commit message: fixed typo

File: catkin_ws/src/my_robot/urdf/my_robot.xacro (robot description, xacro)
@@ -60,6 +60,5 @@
           <origin xyz="0 0 0" rpy="0 1.5707 1.5707"/>
 <mass value="5"/>
-          <inertia> ixx="0.1" ixy="0" ixz="0" iyy="0.1" iyz="0" izz="0.1"
-          </inertia>
+          <inertia ixx="0.1" ixy="0" ixz="0" iyy="0.1" iyz="0" izz="0.1" />
         </internal>
       </link>
@@ -72,6 +71,5 @@
               <origin xyz="0 0 0" rpy="0 1.5707 1.5707"/>
               <mass value="5"/>
-              <inertia> ixx="0.1" ixy="0" ixz="0" iyy="0.1" iyz="0" izz="0.1"
-              </inertia>
+              <inertia> ixx="0.1" ixy="0" ixz="0" iyy="0.1" iyz="0" izz="0.1" />
             </inertial>
           </link>

Commit message: bugfixing

File: catkin_ws/src/my_robot/urdf/my_robot.xacro (robot description, xacro)
@@ -63,30 +63,3 @@
         </internal>
       </link>
-      <link name='right_wheel'>
-        <geometry>
-          <cyclinder radius="0.1" length="0.05">
-          </geometry>
-          <origin>
-            <inertial>
-              <origin xyz="0 0 0" rpy="0 1.5707 1.5707"/>
-              <mass value="5"/>
-              <inertia> ixx="0.1" ixy="0" ixz="0" iyy="0.1" iyz="0" izz="0.1" />
-            </inertial>
-          </link>
-          <joint type="continuous" name="left_wheel_hinge">
-            <origin xyz="0 0.15 0" rpy="0 0 0"/>
-            <child link="left_wheel"/>
-            <parent link="chassis"/>
-            <axis xyz="0 1 0" rpy="0 0 0"/>
-            <limit effort="10000" velocity="1000"/>
-            <dynamics damping="1.0" friction="1.0"/>
-          </joint>
-          <joint type="continuous" name="right_wheel_hinge">
-            <origin xyz="0 0.15 0" rpy="0 0 0"/>
-            <child link="right_wheel"/>
-            <parent link="chassis"/>
-            <axis xyz="0 1 0" rpy="0 0 0"/>
-            <limit effort="10000" velocity="1000"/>
-            <dynamics damping="1.0" friction="1.0"/>
-          </joint>
-        </robot>
+</robot>

Commit message: fixed typo

File: catkin_ws/src/my_robot/urdf/my_robot.xacro (robot description, xacro)
@@ -54,12 +54,39 @@
   <link name='left_wheel'>
     <geometry>
-      <cyclinder radius="0.1" length="0.05">
+      <cyclinder radius="0.1" length="0.05" />
       </geometry>
       <origin>
         <inertial>
           <origin xyz="0 0 0" rpy="0 1.5707 1.5707"/>
-<mass value="5"/>
+          <mass value="5"/>
           <inertia ixx="0.1" ixy="0" ixz="0" iyy="0.1" iyz="0" izz="0.1" />
         </internal>
       </link>
-</robot>
+      <link name='right_wheel'>
+        <geometry>
+          <cyclinder radius="0.1" length="0.05">
+          </geometry>
+          <origin>
+            <inertial>
+              <origin xyz="0 0 0" rpy="0 1.5707 1.5707"/>
+              <mass value="5"/>
+              <inertia> ixx="0.1" ixy="0" ixz="0" iyy="0.1" iyz="0" izz="0.1"/>
+              </inertial>
+            </link>
+            <joint type="continuous" name="left_wheel_hinge">
+              <origin xyz="0 0.15 0" rpy="0 0 0"/>
+              <child link="left_wheel"/>
+              <parent link="chassis"/>
+              <axis xyz="0 1 0" rpy="0 0 0"/>
+              <limit effort="10000" velocity="1000"/>
+              <dynamics damping="1.0" friction="1.0"/>
+            </joint>
+            <joint type="continuous" name="right_wheel_hinge">
+              <origin xyz="0 0.15 0" rpy="0 0 0"/>
+              <child link="right_wheel"/>
+              <parent link="chassis"/>
+              <axis xyz="0 1 0" rpy="0 0 0"/>
+              <limit effort="10000" velocity="1000"/>
+              <dynamics damping="1.0" friction="1.0"/>
+            </joint>
+          </robot>

Commit message: double origin lines

File: catkin_ws/src/my_robot/urdf/my_robot.xacro (robot description, xacro)
@@ -56,5 +56,4 @@
       <cyclinder radius="0.1" length="0.05" />
       </geometry>
-      <origin>
         <inertial>
           <origin xyz="0 0 0" rpy="0 1.5707 1.5707"/>
@@ -67,5 +66,4 @@
           <cyclinder radius="0.1" length="0.05">
           </geometry>
-          <origin>
             <inertial>
               <origin xyz="0 0 0" rpy="0 1.5707 1.5707"/>

Commit message: typos fixed

File: catkin_ws/src/my_robot/urdf/my_robot.xacro (robot description, xacro)
@@ -60,9 +60,9 @@
           <mass value="5"/>
           <inertia ixx="0.1" ixy="0" ixz="0" iyy="0.1" iyz="0" izz="0.1" />
-        </internal>
+        </inertial>
       </link>
       <link name='right_wheel'>
         <geometry>
-          <cyclinder radius="0.1" length="0.05">
+          <cyclinder radius="0.1" length="0.05"/>
           </geometry>
             <inertial>

Commit message: removed obsolte ">"

File: catkin_ws/src/my_robot/urdf/my_robot.xacro (robot description, xacro)
@@ -69,5 +69,5 @@
               <origin xyz="0 0 0" rpy="0 1.5707 1.5707"/>
               <mass value="5"/>
-              <inertia> ixx="0.1" ixy="0" ixz="0" iyy="0.1" iyz="0" izz="0.1"/>
+              <inertia ixx="0.1" ixy="0" ixz="0" iyy="0.1" iyz="0" izz="0.1"/>
               </inertial>
             </link>

Commit message: removed right wheel and joint

File: catkin_ws/src/my_robot/urdf/my_robot.xacro (robot description, xacro)
@@ -62,4 +62,13 @@
         </inertial>
       </link>
+        <joint type="continuous" name="left_wheel_hinge">
+              <origin xyz="0 0.15 0" rpy="0 0 0"/>
+              <child link="left_wheel"/>
+              <parent link="chassis"/>
+              <axis xyz="0 1 0" rpy="0 0 0"/>
+              <limit effort="10000" velocity="1000"/>
+              <dynamics damping="1.0" friction="1.0"/>
+            </joint>
+<!--
       <link name='right_wheel'>
         <geometry>
@@ -72,12 +81,4 @@
               </inertial>
             </link>
-            <joint type="continuous" name="left_wheel_hinge">
-              <origin xyz="0 0.15 0" rpy="0 0 0"/>
-              <child link="left_wheel"/>
-              <parent link="chassis"/>
-              <axis xyz="0 1 0" rpy="0 0 0"/>
-              <limit effort="10000" velocity="1000"/>
-              <dynamics damping="1.0" friction="1.0"/>
-            </joint>
             <joint type="continuous" name="right_wheel_hinge">
               <origin xyz="0 0.15 0" rpy="0 0 0"/>
@@ -88,3 +89,4 @@
               <dynamics damping="1.0" friction="1.0"/>
             </joint>
+-->
           </robot>

Commit message: remove dintertial tag

File: catkin_ws/src/my_robot/urdf/my_robot.xacro (robot description, xacro)
@@ -52,15 +52,13 @@
     </visual>
   </link>
-<!--
   <link name='left_wheel'>
     <geometry>
       <cyclinder radius="0.1" length="0.05" />
       </geometry>
-        <inertial>
           <origin xyz="0 0 0" rpy="0 1.5707 1.5707"/>
           <mass value="5"/>
           <inertia ixx="0.1" ixy="0" ixz="0" iyy="0.1" iyz="0" izz="0.1" />
-        </inertial>
       </link>
+<!--
         <joint type="continuous" name="left_wheel_hinge">
               <origin xyz="0 0.15 0" rpy="0 0 0"/>

Commit message: added inertial, visdual, colision to left wheel

File: catkin_ws/src/my_robot/urdf/my_robot.xacro (robot description, xacro)
@@ -53,10 +53,45 @@
   </link>
   <link name='left_wheel'>
-    <geometry>
-      <cyclinder radius="0.1" length="0.05" />
+     <inertial>
+      <origin xyz="0 0 0" rpy="0 1.5707 1.5707"/>
+      <mass value="5"/>
+        <geometry>
+          <cyclinder radius="0.1" length="0.05" />
+        </geometry>
+        <inertia ixx="0.1" ixy="0" ixz="0" iyy="0.1" iyz="0" izz="0.1" />
+      </inertial>
+   <visual>
+      <origin xyz="0 0 0" rpy="0 1.5707 1.5707"/>
+      <mass value="5"/>
+        <geometry>
+          <cyclinder radius="0.1" length="0.05" />
+        </geometry>
+        <inertia ixx="0.1" ixy="0" ixz="0" iyy="0.1" iyz="0" izz="0.1" />
+      </visual>
+    <collision>
+      <origin xyz="0 0 0" rpy="0 1.5707 1.5707"/>
+      <mass value="5"/>
+        <geometry>
+          <cyclinder radius="0.1" length="0.05" />
+        </geometry>
+        <inertia ixx="0.1" ixy="0" ixz="0" iyy="0.1" iyz="0" izz="0.1" />
+      </collision>
+    <inertial>
+      <mass value="15.0"/>
+      <origin xyz="0.0 0 0" rpy=" 0 0 0"/>
+      <inertia ixx="0.1" ixy="0" ixz="0" iyy="0.1" iyz="0" izz="0.1" />
+    </inertial>
+    <collision name='collision'>
+      <origin xyz="0 0 0" rpy=" 0 0 0"/>
+      <geometry>
+        <box size=".4 .2 .1"/>
       </geometry>
-          <origin xyz="0 0 0" rpy="0 1.5707 1.5707"/>
-          <mass value="5"/>
-          <inertia ixx="0.1" ixy="0" ixz="0" iyy="0.1" iyz="0" izz="0.1" />
+    </collision>
+    <visual name='chassis_visual'>
+      <origin xyz="0 0 0" rpy=" 0 0 0"/>
+      <geometry>
+        <box size=".4 .2 .1"/>
+      </geometry>
+    </visual>
       </link>
 <!--

Commit message: Reviewed initial parameters

File: catkin_ws/src/my_robot/urdf/my_robot.xacro (robot description, xacro)
@@ -1,5 +1,4 @@
 <?xml version='1.0'?>
-<robot name="my_robot"
-  xmlns:xacro="http://www.ros.org/wiki/xacro">
+<robot name="my_robot" xmlns:xacro="http://www.ros.org/wiki/xacro">
   <link name="robot_footprint"></link>
   <joint name="robot_footprint_joint" type="fixed">
@@ -13,5 +12,9 @@
       <mass value="15.0"/>
       <origin xyz="0.0 0 0" rpy=" 0 0 0"/>
-      <inertia ixx="0.1" ixy="0" ixz="0" iyy="0.1" iyz="0" izz="0.1" />
+      <inertia
+          ixx="0.1" ixy="0" ixz="0"
+          iyy="0.1" iyz="0"
+          izz="0.1"
+      />
     </inertial>
     <collision name='collision'>
@@ -52,76 +55,3 @@
     </visual>
   </link>
-  <link name='left_wheel'>
-     <inertial>
-      <origin xyz="0 0 0" rpy="0 1.5707 1.5707"/>
-      <mass value="5"/>
-        <geometry>
-          <cyclinder radius="0.1" length="0.05" />
-        </geometry>
-        <inertia ixx="0.1" ixy="0" ixz="0" iyy="0.1" iyz="0" izz="0.1" />
-      </inertial>
-   <visual>
-      <origin xyz="0 0 0" rpy="0 1.5707 1.5707"/>
-      <mass value="5"/>
-        <geometry>
-          <cyclinder radius="0.1" length="0.05" />
-        </geometry>
-        <inertia ixx="0.1" ixy="0" ixz="0" iyy="0.1" iyz="0" izz="0.1" />
-      </visual>
-    <collision>
-      <origin xyz="0 0 0" rpy="0 1.5707 1.5707"/>
-      <mass value="5"/>
-        <geometry>
-          <cyclinder radius="0.1" length="0.05" />
-        </geometry>
-        <inertia ixx="0.1" ixy="0" ixz="0" iyy="0.1" iyz="0" izz="0.1" />
-      </collision>
-    <inertial>
-      <mass value="15.0"/>
-      <origin xyz="0.0 0 0" rpy=" 0 0 0"/>
-      <inertia ixx="0.1" ixy="0" ixz="0" iyy="0.1" iyz="0" izz="0.1" />
-    </inertial>
-    <collision name='collision'>
-      <origin xyz="0 0 0" rpy=" 0 0 0"/>
-      <geometry>
-        <box size=".4 .2 .1"/>
-      </geometry>
-    </collision>
-    <visual name='chassis_visual'>
-      <origin xyz="0 0 0" rpy=" 0 0 0"/>
-      <geometry>
-        <box size=".4 .2 .1"/>
-      </geometry>
-    </visual>
-      </link>
-<!--
-        <joint type="continuous" name="left_wheel_hinge">
-              <origin xyz="0 0.15 0" rpy="0 0 0"/>
-              <child link="left_wheel"/>
-              <parent link="chassis"/>
-              <axis xyz="0 1 0" rpy="0 0 0"/>
-              <limit effort="10000" velocity="1000"/>
-              <dynamics damping="1.0" friction="1.0"/>
-            </joint>
--->
-<!--
-      <link name='right_wheel'>
-        <geometry>
-          <cyclinder radius="0.1" length="0.05"/>
-          </geometry>
-            <inertial>
-              <origin xyz="0 0 0" rpy="0 1.5707 1.5707"/>
-              <mass value="5"/>
-              <inertia ixx="0.1" ixy="0" ixz="0" iyy="0.1" iyz="0" izz="0.1"/>
-              </inertial>
-            </link>
-            <joint type="continuous" name="right_wheel_hinge">
-              <origin xyz="0 0.15 0" rpy="0 0 0"/>
-              <child link="right_wheel"/>
-              <parent link="chassis"/>
-              <axis xyz="0 1 0" rpy="0 0 0"/>
-              <limit effort="10000" velocity="1000"/>
-              <dynamics damping="1.0" friction="1.0"/>
-            </joint>
--->
-          </robot>
+</robot>

Commit message: added left and right wheel and left wheel joint

File: catkin_ws/src/my_robot/urdf/my_robot.xacro (robot description, xacro)
@@ -55,3 +55,63 @@
     </visual>
   </link>
+<!-- definition of wheels -->
+<!-- left wheel, once ready this will be coned to right weel -->
+  <link name='left_wheel'>
+    <pose>0 0 0.1 0 0 0</pose>
+    <inertial>
+      <mass value="5.0"/>
+      <origin xyz="0 0 0" rpy=" 0 1.5707 1.5707"/>
+      <inertia
+          ixx="0.1" ixy="0" ixz="0"
+          iyy="0.1" iyz="0"
+          izz="0.1"
+      />
+    </inertial>
+    <collision name='left_wheel_collision'>
+      <origin xyz="0 0 0" rpy=" 0 1.5707 1.5707"/>
+      <geometry>
+        <cyclinder size="0.1 0.05"/>
+      </geometry>
+    </collision>
+    <visual name='left_wheel_visual'>
+      <origin xyz="0 0 0" rpy=" 0 1.5707 1.5707"/>
+      <geometry>
+        <cyclinder size="0.1 0.05"/>
+      </geometry>
+    </visual>
+  </link>
+<!-- the right wheel-->
+<link name='right_wheel'>
+    <pose>0 0 0.1 0 0 0</pose>
+    <inertial>
+      <mass value="5.0"/>
+      <origin xyz="0 0 0" rpy=" 0 1.5707 1.5707"/>
+      <inertia
+          ixx="0.1" ixy="0" ixz="0"
+          iyy="0.1" iyz="0"
+          izz="0.1"
+      />
+    </inertial>
+    <collision name='right_wheel_collision'>
+      <origin xyz="0 0 0" rpy=" 0 1.5707 1.5707"/>
+      <geometry>
+        <cyclinder size="0.1 0.05"/>
+      </geometry>
+    </collision>
+    <visual name='right_wheel_visual'>
+      <origin xyz="0 0 0" rpy=" 0 1.5707 1.5707"/>
+      <geometry>
+        <cyclinder size="0.1 0.05"/>
+      </geometry>
+    </visual>
+  </link>
+<!-- added joint for the left wheel -->
+  <joint type="continuous" name="left_wheel_hinge">
+    <origin xyz="0 0.15 0" rpy="0 0 0"/>
+    <child link="left_wheel"/>
+    <parent link="chassis"/>
+    <axis xyz="0 1 0" rpy="0 0 0"/>
+    <limit effort="10000" velocity="1000"/>
+    <dynamics damping="1.0" friction="1.0"/>
+  </joint>
 </robot>

Commit message: Changed typo: cyclinder --> cylinder

File: catkin_ws/src/my_robot/urdf/my_robot.xacro (robot description, xacro)
@@ -71,5 +71,5 @@
       <origin xyz="0 0 0" rpy=" 0 1.5707 1.5707"/>
       <geometry>
-        <cyclinder length="0.1" radius="0.05"/>
+        <cylinder length="0.1" radius="0.05"/>
       </geometry>
     </collision>
@@ -77,5 +77,5 @@
       <origin xyz="0 0 0" rpy=" 0 1.5707 1.5707"/>
       <geometry>
-         <cyclinder length="0.1" radius="0.05"/>
+         <cylinder length="0.1" radius="0.05"/>
       </geometry>
     </visual>
@@ -96,5 +96,5 @@
       <origin xyz="0 0 0" rpy=" 0 1.5707 1.5707"/>
       <geometry>
-         <cyclinder length="0.1" radius="0.05"/>
+         <cylinder length="0.1" radius="0.05"/>
       </geometry>
     </collision>
@@ -102,5 +102,5 @@
       <origin xyz="0 0 0" rpy=" 0 1.5707 1.5707"/>
       <geometry>
-         <cyclinder length="0.1" radius="0.05"/>
+         <cylinder length="0.1" radius="0.05"/>
       </geometry>
     </visual>

Commit message: test add of right join to

File: catkin_ws/src/my_robot/urdf/my_robot.xacro (robot description, xacro)
@@ -115,3 +115,12 @@
     <dynamics damping="1.0" friction="1.0"/>
   </joint>
+!-- added joint for the left wheel -->
+  <joint type="continuous" name="right_wheel_hinge">
+    <origin xyz="0 0.15 0" rpy="0 0 0"/>
+    <child link="right_wheel"/>
+    <parent link="chassis"/>
+    <axis xyz="0 1 0" rpy="0 0 0"/>
+    <limit effort="10000" velocity="1000"/>
+    <dynamics damping="1.0" friction="1.0"/>
+  </joint>
 </robot>

Commit message: removed join for debugging

File: catkin_ws/src/my_robot/urdf/my_robot.xacro (robot description, xacro)
@@ -107,5 +107,5 @@
   </link>
 <!-- added joint for the left wheel -->
-  <joint type="continuous" name="left_wheel_hinge">
+<!--   <joint type="continuous" name="left_wheel_hinge">
     <origin xyz="0 0.15 0" rpy="0 0 0"/>
     <child link="left_wheel"/>
@@ -115,12 +115,4 @@
     <dynamics damping="1.0" friction="1.0"/>
   </joint>
-!-- added joint for the left wheel -->
-  <joint type="continuous" name="right_wheel_hinge">
-    <origin xyz="0 0.15 0" rpy="0 0 0"/>
-    <child link="right_wheel"/>
-    <parent link="chassis"/>
-    <axis xyz="0 1 0" rpy="0 0 0"/>
-    <limit effort="10000" velocity="1000"/>
-    <dynamics damping="1.0" friction="1.0"/>
-  </joint>
+-->
 </robot>

Commit message: new definition of front left and fron right wheel

File: catkin_ws/src/my_robot/urdf/my_robot.xacro (robot description, xacro)
@@ -55,64 +55,43 @@
     </visual>
   </link>
-<!-- definition of wheels -->
-<!-- left wheel, once ready this will be coned to right weel -->
-  <link name='left_wheel'>
-    <pose>0 0 0.1 0 0 0</pose>
-    <inertial>
-      <mass value="5.0"/>
-      <origin xyz="0 0 0" rpy=" 0 1.5707 1.5707"/>
-      <inertia
-          ixx="0.1" ixy="0" ixz="0"
-          iyy="0.1" iyz="0"
-          izz="0.1"
-      />
-    </inertial>
-    <collision name='left_wheel_collision'>
-      <origin xyz="0 0 0" rpy=" 0 1.5707 1.5707"/>
-      <geometry>
-        <cylinder length="0.1" radius="0.05"/>
-      </geometry>
-    </collision>
-    <visual name='left_wheel_visual'>
-      <origin xyz="0 0 0" rpy=" 0 1.5707 1.5707"/>
-      <geometry>
-         <cylinder length="0.1" radius="0.05"/>
-      </geometry>
-    </visual>
-  </link>
-<!-- the right wheel-->
-<link name='right_wheel'>
-    <pose>0 0 0.1 0 0 0</pose>
-    <inertial>
-      <mass value="5.0"/>
-      <origin xyz="0 0 0" rpy=" 0 1.5707 1.5707"/>
-      <inertia
-          ixx="0.1" ixy="0" ixz="0"
-          iyy="0.1" iyz="0"
-          izz="0.1"
-      />
-    </inertial>
-    <collision name='right_wheel_collision'>
-      <origin xyz="0 0 0" rpy=" 0 1.5707 1.5707"/>
-      <geometry>
-         <cylinder length="0.1" radius="0.05"/>
-      </geometry>
-    </collision>
-    <visual name='right_wheel_visual'>
-      <origin xyz="0 0 0" rpy=" 0 1.5707 1.5707"/>
-      <geometry>
-         <cylinder length="0.1" radius="0.05"/>
-      </geometry>
-    </visual>
-  </link>
-<!-- added joint for the left wheel -->
-<!--   <joint type="continuous" name="left_wheel_hinge">
-    <origin xyz="0 0.15 0" rpy="0 0 0"/>
-    <child link="left_wheel"/>
-    <parent link="chassis"/>
-    <axis xyz="0 1 0" rpy="0 0 0"/>
-    <limit effort="10000" velocity="1000"/>
-    <dynamics damping="1.0" friction="1.0"/>
-  </joint>
--->
+<!-- Right Front Wheel -->
+	<link name="front_right_wheel">
+		<visual>
+			<origin xyz="0 0 0" rpy=" 0 1.5707 1.5707" />
+			<geometry>
+				<cylinder radius="0.1" length="0.05" />
+			</geometry>
+		</visual>
+		<collision>
+			<origin xyz="0 0 0" rpy=" 0 1.5707 1.5707" />
+			<geometry>
+				<cylinder radius="0.1" length="0.05" />
+			</geometry>
+		</collision>
+		<inertial>
+			<mass value="5.0" />
+			<origin xyz="0 0 0" rpy=" 0 1.5707 1.5707" />
+			<inertia ixx="0.1" ixy="0" ixz="0" iyy="0.1" iyz="0" izz="0.1" />
+		</inertial>
+	</link>
+  <!-- Left Front Wheel -->
+	<link name="front_left_wheel">
+		<visual>
+			<origin xyz="0 0 0" rpy=" 0 1.5707 1.5707" />
+			<geometry>
+				<cylinder radius="0.1" length="0.05" />
+			</geometry>
+		</visual>
+		<collision>
+			<origin xyz="0 0 0" rpy=" 0 1.5707 1.5707" />
+			<geometry>
+				<cylinder radius="0.1" length="0.05" />
+			</geometry>
+		</collision>
+		<inertial>
+			<mass value="5.0" />
+			<origin xyz="0 0 0" rpy=" 0 1.5707 1.5707" />
+			<inertia ixx="0.1" ixy="0" ixz="0" iyy="0.1" iyz="0" izz="0.1" />
+		</inertial>
+	</link>
 </robot>
