Commit message: Added left joint

File: catkin_ws/src/my_robot/urdf/my_robot.xacro (robot description, xacro)
@@ -55,6 +55,6 @@
     </visual>
   </link>
-<!-- Right Front Wheel -->
-	<link name="front_right_wheel">
+<!-- Right Wheel -->
+	<link name="right_wheel">
 		<visual>
 			<origin xyz="0 0 0" rpy=" 0 1.5707 1.5707" />
@@ -75,6 +75,6 @@
 		</inertial>
 	</link>
-  <!-- Left Front Wheel -->
-	<link name="front_left_wheel">
+  <!-- Front Wheel -->
+	<link name="left_wheel">
 		<visual>
 			<origin xyz="0 0 0" rpy=" 0 1.5707 1.5707" />
@@ -95,3 +95,11 @@
 		</inertial>
 	</link>
+  <joint type="continuous" name="left_wheel_hinge">
+    <origin xyz="0 0.15 0" rpy="0 0 0"/>
+    <child link="left_wheel"/>
+    <parent link="chassis"/>
+    <axis xyz="0 1 0" rpy="0 0 0"/>
+    <limit effort="10000" velocity="1000"/>
+    <dynamics damping="1.0" friction="1.0"/>
+  </joint>
 </robot>

Commit message: Added right joint

File: catkin_ws/src/my_robot/urdf/my_robot.xacro (robot description, xacro)
@@ -95,4 +95,5 @@
 		</inertial>
 	</link>
+<!-- Joint left wheel -->
   <joint type="continuous" name="left_wheel_hinge">
     <origin xyz="0 0.15 0" rpy="0 0 0"/>
@@ -103,3 +104,12 @@
     <dynamics damping="1.0" friction="1.0"/>
   </joint>
+<!-- Joint left wheel -->
+  <joint type="continuous" name="right_wheel_hinge">
+    <origin xyz="0 0.15 0" rpy="0 0 0"/>
+    <child link="right_wheel"/>
+    <parent link="chassis"/>
+    <axis xyz="0 1 0" rpy="0 0 0"/>
+    <limit effort="10000" velocity="1000"/>
+    <dynamics damping="1.0" friction="1.0"/>
+  </joint>
 </robot>

Commit message: fixed joint offset

File: catkin_ws/src/my_robot/urdf/my_robot.xacro (robot description, xacro)
@@ -75,5 +75,5 @@
 		</inertial>
 	</link>
-  <!-- Front Wheel -->
+  <!-- Left Wheel -->
 	<link name="left_wheel">
 		<visual>
@@ -106,5 +106,5 @@
 <!-- Joint left wheel -->
   <joint type="continuous" name="right_wheel_hinge">
-    <origin xyz="0 0.15 0" rpy="0 0 0"/>
+    <origin xyz="0 -0.15 0" rpy="0 0 0"/>
     <child link="right_wheel"/>
     <parent link="chassis"/>

Commit message: added Camera, LIDAR and mesh

File: catkin_ws/src/my_robot/urdf/my_robot.xacro (robot description, xacro)
@@ -113,3 +113,55 @@
     <dynamics damping="1.0" friction="1.0"/>
   </joint>
+<!-- Camera Link & Joint -->
+	<link name="camera">
+		<visual>
+			<origin xyz="-0.0 0 0" rpy=" 0 0 0" />
+			<geometry>
+				<box size="0.05 0.05 0.05" />
+			</geometry>
+		</visual>
+		<collision>
+			<origin xyz="-0.0 0 0" rpy=" 0 0 0" />
+			<geometry>
+				<box size="0.05 0.05 0.05" />
+			</geometry>
+		</collision>
+		<inertial>
+			<mass value="0.1" />
+			<origin xyz="0.0 0 0" rpy=" 0 0 0" />
+			<inertia ixx="1e-6" ixy="0" ixz="0" iyy="1e-6" iyz="0" izz="1e-6" />
+		</inertial>
+	</link>
+	<joint type="fixed" name="camera_joint">
+		<origin xyz="0.4 0 0" rpy="0 0 0" />
+		<child link="camera" />
+		<parent link="chassis" />
+		<axis xyz="0 1 0" rpy="0 0 0" />
+	</joint>
+  <!-- LIDAR Link & Joint -->
+	<link name="hokuyo">
+		<visual>
+			<origin xyz="-0.0 0 0" rpy=" 0 0 0" />
+			<geometry>
+				<mesh filename="package://go_chase_it/meshes/hokuyo.dae" />
+			</geometry>
+		</visual>
+		<collision>
+			<origin xyz="-0.0 0 0" rpy=" 0 0 0" />
+			<geometry>
+				<box size="0.01 0.01 0.01" />
+			</geometry>
+		</collision>
+		<inertial>
+			<mass value="1e-5" />
+			<origin xyz="0.0 0 0" rpy=" 0 0 0" />
+			<inertia ixx="1e-6" ixy="0" ixz="0" iyy="1e-6" iyz="0" izz="1e-6" />
+		</inertial>
+	</link>
+	<joint type="fixed" name="hokuyo">
+		<origin xyz="0.35 0 0.1" rpy="0 0 0" />
+		<child link="hokuyo" />
+		<parent link="chassis" />
+		<axis xyz="0 1 0" rpy="0 0 0" />
+	</joint>
 </robot>

Commit message: fixed wrong package path

File: catkin_ws/src/my_robot/urdf/my_robot.xacro (robot description, xacro)
@@ -144,5 +144,5 @@
 			<origin xyz="-0.0 0 0" rpy=" 0 0 0" />
 			<geometry>
-				<mesh filename="package://go_chase_it/meshes/hokuyo.dae" />
+				<mesh filename="package://my_robot/meshes/hokuyo.dae" />
 			</geometry>
 		</visual>

Commit message: adapted origins

File: catkin_ws/src/my_robot/urdf/my_robot.xacro (robot description, xacro)
@@ -134,5 +134,5 @@
 	</link>
 	<joint type="fixed" name="camera_joint">
-		<origin xyz="0.4 0 0" rpy="0 0 0" />
+		<origin xyz="0.2 0 0" rpy="0 0 0" />
 		<child link="camera" />
 		<parent link="chassis" />
@@ -142,5 +142,5 @@
 	<link name="hokuyo">
 		<visual>
-			<origin xyz="-0.0 0 0" rpy=" 0 0 0" />
+			<origin xyz="0 0 0" rpy=" 0 0 0" />
 			<geometry>
 				<mesh filename="package://my_robot/meshes/hokuyo.dae" />
@@ -148,17 +148,17 @@
 		</visual>
 		<collision>
-			<origin xyz="-0.0 0 0" rpy=" 0 0 0" />
+			<origin xyz="-0 0 0" rpy=" 0 0 0" />
 			<geometry>
-				<box size="0.01 0.01 0.01" />
+				<box size="0.1 0.1 0.1" />
 			</geometry>
 		</collision>
 		<inertial>
 			<mass value="1e-5" />
-			<origin xyz="0.0 0 0" rpy=" 0 0 0" />
+			<origin xyz="0.15 0 0.1" rpy=" 0 0 0" />
 			<inertia ixx="1e-6" ixy="0" ixz="0" iyy="1e-6" iyz="0" izz="1e-6" />
 		</inertial>
 	</link>
 	<joint type="fixed" name="hokuyo">
-		<origin xyz="0.35 0 0.1" rpy="0 0 0" />
+		<origin xyz="0.15 0 0.1" rpy="0 0 0" />
 		<child link="hokuyo" />
 		<parent link="chassis" />

Commit message: added Material to both wheels and chassis

File: catkin_ws/src/my_robot/urdf/my_robot.xacro (robot description, xacro)
@@ -55,4 +55,7 @@
     </visual>
   </link>
+  <gazebo reference="chassis">
+    <material>Gazebo/Green</material>
+  </gazebo>
 <!-- Right Wheel -->
 	<link name="right_wheel">
@@ -75,4 +78,7 @@
 		</inertial>
 	</link>
+  <gazebo reference="right_wheel">
+    <material>Gazebo/Blue</material>
+  </gazebo>
   <!-- Left Wheel -->
 	<link name="left_wheel">
@@ -95,4 +101,7 @@
 		</inertial>
 	</link>
+  <gazebo reference="left_wheel">
+    <material>Gazebo/Blue</material>
+  </gazebo>
 <!-- Joint left wheel -->
   <joint type="continuous" name="left_wheel_hinge">
